Commit message: working very clsoe already

File: aic_assets/models/Basler Camera/basler_camera_macro.xacro (robot description, xacro)
@@ -93,4 +93,64 @@
           </camera>
         </sensor>
+        <sensor name="${name}_segmentation" type="segmentation_camera">
+          <pose>0 0 0 0 0 0</pose>
+          <update_rate>20.0</update_rate>
+          <topic>/${name}/segmentation</topic>
+          <always_on>true</always_on>
+          <frame_id>${tf_prefix}sensor_link</frame_id>
+          <camera name="${name}_segmentation">
+            <optical_frame_id>${tf_prefix}optical</optical_frame_id>
+            <image>
+              <width>1152</width>
+              <height>1024</height>
+            </image>
+            <horizontal_fov>0.8718</horizontal_fov>
+            <clip>
+              <near>0.07</near>
+              <far>20</far>
+            </clip>
+            <segmentation_type>instance</segmentation_type>
+          </camera>
+        </sensor>
+        <sensor name="${name}_bbox" type="boundingbox_camera">
+          <pose>0 0 0 0 0 0</pose>
+          <update_rate>20.0</update_rate>
+          <topic>/${name}/bounding_boxes</topic>
+          <always_on>true</always_on>
+          <frame_id>${tf_prefix}sensor_link</frame_id>
+          <camera name="${name}_bbox">
+            <box_type>visible_2d</box_type>
+            <optical_frame_id>${tf_prefix}optical</optical_frame_id>
+            <image>
+              <width>1152</width>
+              <height>1024</height>
+            </image>
+            <horizontal_fov>0.8718</horizontal_fov>
+            <clip>
+              <near>0.07</near>
+              <far>20</far>
+            </clip>
+          </camera>
+        </sensor>
+        <sensor name="${name}_depth" type="depth_camera">
+          <pose>0 0 0 0 0 0</pose>
+          <update_rate>20.0</update_rate>
+          <topic>/${name}/depth</topic>
+          <always_on>true</always_on>
+          <frame_id>${tf_prefix}sensor_link</frame_id>
+          <camera name="${name}_depth">
+            <camera_info_topic>/${name}/depth/camera_info</camera_info_topic>
+            <optical_frame_id>${tf_prefix}optical</optical_frame_id>
+            <image>
+              <width>1152</width>
+              <height>1024</height>
+            </image>
+            <horizontal_fov>0.8718</horizontal_fov>
+            <clip>
+              <near>0.07</near>
+              <far>20</far>
+            </clip>
+          </camera>
+        </sensor>
       </gazebo>
     </xacro:if>

File: aic_assets/models/NIC Card Mount/nic_card_mount_macro.xacro (robot description, xacro)
@@ -1,5 +1,5 @@
 <?xml version="1.0" ?>
 <robot xmlns:xacro="http://wiki.ros.org/xacro">
-  <xacro:macro name="nic_card_mount" params="prefix pose">
+  <xacro:macro name="nic_card_mount" params="prefix pose bbox_label:=10">
     <gazebo>
       <include>
@@ -25,4 +25,7 @@
           <collision>contact_collision_02</collision>
         </plugin>
+        <plugin filename="gz-sim-label-system" name="gz::sim::systems::Label">
+          <label>${bbox_label}</label>
+        </plugin>
       </include>
     </gazebo>

File: aic_assets/models/SC Port/sc_port_macro.xacro (robot description, xacro)
@@ -1,5 +1,5 @@
 <?xml version="1.0" ?>
 <robot xmlns:xacro="http://wiki.ros.org/xacro">
-  <xacro:macro name="sc_port" params="prefix pose">
+  <xacro:macro name="sc_port" params="prefix pose bbox_label:=20">
     <gazebo>
       <include>
@@ -15,4 +15,7 @@
           <enabled>true</enabled>
         </plugin>
+        <plugin filename="gz-sim-label-system" name="gz::sim::systems::Label">
+          <label>${bbox_label}</label>
+        </plugin>
       </include>
     </gazebo>
